File: omega-dock-new.sch (KiCad schematic (older format))
At the start: 18 parts, among them J1 USB_A, J2 USB_PWR, J3 RJ45-TRAFO, U1 USBLC6-2, U2 AP111733, U3 OMEGA_2

Commit message: ajustando a kicad 5
Parts:
- C1, C2: symbol CP_Small -> omega-dock-new-rescue:CP_Small-RESCUE-omega-dock-new
- C3, C4, C5: symbol C -> omega-dock-new-rescue:C-RESCUE-omega-dock-new
- D1: symbol LED -> omega-dock-new-rescue:LED-RESCUE-omega-dock-new
- F1: symbol Polyfuse -> omega-dock-new-rescue:Polyfuse-RESCUE-omega-dock-new
- J1: symbol USB_A -> omega-dock-new-rescue:USB_A-RESCUE-omega-dock-new
- J2: symbol USB_OTG -> omega-dock-new-rescue:USB_OTG-RESCUE-omega-dock-new
- J3: symbol RJ45-TRAFO -> omega-dock-new:RJ45-TRAFO
- R1, R2, R3, R4, R5: symbol R -> omega-dock-new-rescue:R-RESCUE-omega-dock-new
- U1: symbol USBLC6-2 -> omega-dock-new:USBLC6-2
- U2: symbol AP111733 -> omega-dock-new-rescue:AP111733-RESCUE-omega-dock-new
- U3: symbol OMEGA_2 -> omega-dock-new:OMEGA_2
Connections:
- wire segments 69 -> 80
Changed lines of the file:
@@
-EESchema Schematic File Version 2
-LIBS:power
-LIBS:device
-LIBS:transistors
-LIBS:conn
-LIBS:linear
-LIBS:regul
-LIBS:74xx
-LIBS:cmos4000
-LIBS:adc-dac
-LIBS:memory
-LIBS:xilinx
-LIBS:microcontrollers
-LIBS:dsp
-LIBS:microchip
-LIBS:analog_switches
-LIBS:motorola
-LIBS:texas
-LIBS:intel
-LIBS:audio
-LIBS:interface
-LIBS:digital-audio
-LIBS:philips
-LIBS:display
-LIBS:cypress
-LIBS:siliconi
-LIBS:opto
-LIBS:atmel
-LIBS:contrib
-LIBS:valves
-LIBS:omega-dock-new
+EESchema Schematic File Version 4
 LIBS:omega-dock-new-cache
 EELAYER 26 0
@@
 $EndDescr
 $Comp
-L USB_OTG J2
+L omega-dock-new-rescue:USB_OTG-RESCUE-omega-dock-new J2
 U 1 1 5950B756
 P 1300 3900
@@
 $EndComp
 $Comp
-L USB_A J1
+L omega-dock-new-rescue:USB_A-RESCUE-omega-dock-new J1
 U 1 1 5950B98B
 P 1450 1950
@@
 $EndComp
 $Comp
-L +5V #PWR01
+L power1:+5V #PWR01
 U 1 1 5950BD7E
 P 1800 1450
@@
 $EndComp
 Wire Wire Line
-	1600 3700 2050 3700
+	1600 3700 1750 3700
 Wire Wire Line
 	1750 3700 1750 3600
 $Comp
-L +5V #PWR02
+L power1:+5V #PWR02
 U 1 1 5950C251
 P 1750 3600
@@
 	1200 4300 1300 4300
 $Comp
-L GND #PWR03
+L power1:GND #PWR03
 U 1 1 5950C2F7
 P 1300 4400
@@
 	1650 4000 1600 4000
 Wire Wire Line
-	5500 4850 7350 4850
+	5500 4850 6700 4850
 Wire Wire Line
 	5500 4550 6200 4550
@@
 	7750 4950 7850 4950
 Wire Wire Line
-	7750 3950 7750 4950
+	7750 3950 7750 4650
 Wire Wire Line
 	7750 4650 7850 4650
 Connection ~ 7750 4650
 $Comp
-L C C5
+L omega-dock-new-rescue:C-RESCUE-omega-dock-new C5
 U 1 1 5950E1D8
 P 8050 4150
@@
 $EndComp
 Wire Wire Line
-	7650 3950 8050 3950
+	7650 3950 7750 3950
 Wire Wire Line
 	8050 3950 8050 4000
 Connection ~ 7750 3950
 $Comp
-L GND #PWR04
+L power1:GND #PWR04
 U 1 1 5950E32A
 P 8050 4300
@@
 $EndComp
 $Comp
-L R R1
+L omega-dock-new-rescue:R-RESCUE-omega-dock-new R1
 U 1 1 5950E906
 P 6450 4400
@@
 $EndComp
 $Comp
-L R R2
+L omega-dock-new-rescue:R-RESCUE-omega-dock-new R2
 U 1 1 5950E933
 P 6700 4400
@@
 $EndComp
 $Comp
-L R R3
+L omega-dock-new-rescue:R-RESCUE-omega-dock-new R3
 U 1 1 5950EB0A
 P 6450 5350
@@
 $EndComp
 $Comp
-L R R4
+L omega-dock-new-rescue:R-RESCUE-omega-dock-new R4
 U 1 1 5950EB41
 P 6700 5350
@@
 	6700 5500 6450 5500
 $Comp
-L C C4
+L omega-dock-new-rescue:C-RESCUE-omega-dock-new C4
 U 1 1 5950F143
 P 6700 5700
@@
 $EndComp
 $Comp
-L C C3
+L omega-dock-new-rescue:C-RESCUE-omega-dock-new C3
 U 1 1 5950F19F
 P 6700 4050
@@
 Connection ~ 6700 4250
 $Comp
-L GND #PWR05
+L power1:GND #PWR05
 U 1 1 5950F3FA
 P 6700 3900
@@
 $EndComp
 $Comp
-L GND #PWR06
+L power1:GND #PWR06
 U 1 1 5950F5A6
 P 6700 5850
@@
 	1950 2100 2600 2100
 $Comp
-L GND #PWR07
+L power1:GND #PWR07
 U 1 1 595105A0
 P 2400 2150
@@
 $EndComp
 $Comp
-L +3.3V #PWR08
+L power1:+3.3V #PWR08
 U 1 1 59510668
 P 3650 1650
@@
 	5800 3650 5500 3650
 $Comp
-L AP111733 U2
+L omega-dock-new-rescue:AP111733-RESCUE-omega-dock-new U2
 U 1 1 59510FB8
 P 2350 3700
@@
 Connection ~ 1750 3700
 $Comp
-L CP_Small C1
+L omega-dock-new-rescue:CP_Small-RESCUE-omega-dock-new C1
 U 1 1 59511627
 P 1900 3850
@@
 $EndComp
 $Comp
-L CP_Small C2
+L omega-dock-new-rescue:CP_Small-RESCUE-omega-dock-new C2
 U 1 1 595116AD
 P 2800 3850
@@
 	2650 3700 2800 3700
 $Comp
-L GND #PWR09
+L power1:GND #PWR09
 U 1 1 5951185A
 P 2800 3950
@@
 $EndComp
 $Comp
-L GND #PWR010
+L power1:GND #PWR010
 U 1 1 595118AA
 P 2350 4000
@@
 $EndComp
 $Comp
-L GND #PWR011
+L power1:GND #PWR011
 U 1 1 595118DC
 P 1900 3950
@@
 Connection ~ 1900 3700
 $Comp
-L +3.3V #PWR012
+L power1:+3.3V #PWR012
 U 1 1 59511B86
 P 2800 3600
@@
 $EndComp
 Wire Wire Line
-	2800 3600 2800 3750
+	2800 3600 2800 3700
 Connection ~ 2800 3700
 $Comp
-L GND #PWR013
+L power1:GND #PWR013
 U 1 1 59512193
 P 1450 2500
@@
 $EndComp
 $Comp
-L GND #PWR014
+L power1:GND #PWR014
 U 1 1 59512B28
 P 7600 5750
@@
 	4000 3350 3950 3350
 Wire Wire Line
-	3950 3350 3950 3150
-Wire Wire Line
-	3850 3150 5500 3150
-Wire Wire Line
-	5500 3150 5500 3350
-$Comp
-L GND #PWR015
+	3950 3350 3950 2950
+Wire Wire Line
+	3700 2950 3950 2950
+Wire Wire Line
+	5500 2950 5500 3350
+$Comp
+L power1:GND #PWR015
 U 1 1 595130B7
-P 3850 3200
-F 0 "#PWR015" H 3850 2950 50  0001 C CNN
-F 1 "GND" H 3850 3050 50  0000 C CNN
-F 2 "" H 3850 3200 50  0001 C CNN
-F 3 "" H 3850 3200 50  0001 C CNN
-	1    3850 3200
-	1    0    0    -1
-$EndComp
-$Comp
-L +3.3V #PWR016
+P 3700 3200
+F 0 "#PWR015" H 3700 2950 50  0001 C CNN
+F 1 "GND" H 3700 3050 50  0000 C CNN
+F 2 "" H 3700 3200 50  0001 C CNN
+F 3 "" H 3700 3200 50  0001 C CNN
+	1    3700 3200
+	1    0    0    -1
+$EndComp
+$Comp
+L power1:+3.3V #PWR016
 U 1 1 595130E9
 P 6000 3200
@@
 $EndComp
 Wire Wire Line
-	3850 3150 3850 3200
-Connection ~ 3950 3150
+	3700 2950 3700 3200
+Connection ~ 3950 2950
 NoConn ~ 4000 3500
 NoConn ~ 4000 3650
@@
 	1350 2400 1450 2400
 Wire Wire Line
-	1450 2350 1450 2500
+	1450 2350 1450 2400
 Connection ~ 1450 2400
 Wire Wire Line
@@
 UD-
 $Comp
-L Polyfuse F1
+L omega-dock-new-rescue:Polyfuse-RESCUE-omega-dock-new F1
 U 1 1 5952722D
 P 1800 1600
@@
 	1750 1750 1800 1750
 $Comp
-L USBLC6-2 U1
+L omega-dock-new:USBLC6-2 U1
 U 1 1 5951020C
 P 3050 2000
@@
 $EndComp
 $Comp
-L OMEGA_2 U3
+L omega-dock-new:OMEGA_2 U3
 U 1 1 5952F8F9
 P 4750 4400
@@
 	6300 5550 6300 4200
 $Comp
-L RJ45-TRAFO J3
+L omega-dock-new:RJ45-TRAFO J3
 U 1 1 59867667
 P 9150 5050
@@
 	6200 4550 6200 5050
 Wire Wire Line
-	6200 5050 7850 5050
+	6200 5050 6450 5050
 Wire Wire Line
 	5500 4700 6150 4700
@@
 	6150 4700 6150 5000
 Wire Wire Line
-	6150 5000 7650 5000
+	6150 5000 6700 5000
 Wire Wire Line
 	7650 5000 7650 4850
@@
 	5750 5000 5750 4800
 Wire Wire Line
-	5750 4800 7300 4800
+	5750 4800 6450 4800
 Wire Wire Line
 	7300 4800 7300 4550
@@
 ETH_PWR
 $Comp
-L LED D1
+L omega-dock-new-rescue:LED-RESCUE-omega-dock-new D1
 U 1 1 5986906A
 P 7350 3150
@@
 $EndComp
 $Comp
-L +3.3V #PWR017
+L power1:+3.3V #PWR017
 U 1 1 598696ED
 P 7350 2700
@@
 $EndComp
 $Comp
-L R R5
+L omega-dock-new-rescue:R-RESCUE-omega-dock-new R5
 U 1 1 5986972A
 P 7350 2850
@@
 $EndComp
 $Comp
-L GND #PWR018
+L power1:GND #PWR018
 U 1 1 5986977F
 P 7350 3300
@@
 $EndComp
 NoConn ~ 7850 5250
+Wire Wire Line
+	7750 4650 7750 4950
+Wire Wire Line
+	7750 3950 8050 3950
+Wire Wire Line
+	6700 4850 7350 4850
+Wire Wire Line
+	6450 4800 7300 4800
+Wire Wire Line
+	1750 3700 1900 3700
+Wire Wire Line
+	1900 3700 2050 3700
+Wire Wire Line
+	2800 3700 2800 3750
+Wire Wire Line
+	3950 2950 5500 2950
+Wire Wire Line
+	1450 2400 1450 2500
+Wire Wire Line
+	6450 5050 7850 5050
+Wire Wire Line
+	6700 5000 7650 5000
 $EndSCHEMATC

Commit message: redimencioando unas cosas
Parts:
- removed J2: USB_PWR, Connectors:USB_Micro-B, symbol omega-dock-new-rescue:USB_OTG-RESCUE-omega-dock-new
- added J2: Conn_01x02, Connector_PinHeader_2.54mm:PinHeader_1x02_P2.54mm_Vertical, symbol Connector_Generic:Conn_01x02
Connections:
- net labels added: RX, TX
- wire segments 80 -> 79
- no-connect marks 24 -> 21
Changed lines of the file:
@@
 $EndDescr
-$Comp
-L omega-dock-new-rescue:USB_OTG-RESCUE-omega-dock-new J2
-U 1 1 5950B756
-P 1300 3900
-F 0 "J2" H 1100 4350 50  0000 L CNN
-F 1 "USB_PWR" H 1100 4250 50  0000 L CNN
-F 2 "Connectors:USB_Micro-B" H 1450 3850 50  0001 C CNN
-F 3 "" H 1450 3850 50  0001 C CNN
-	1    1300 3900
-	1    0    0    -1
-$EndComp
 $Comp
 L omega-dock-new-rescue:USB_A-RESCUE-omega-dock-new J1
@@
 $EndComp
 Wire Wire Line
-	1600 3700 1750 3700
+	1450 3700 1750 3700
 Wire Wire Line
 	1750 3700 1750 3600
@@
 $EndComp
 Wire Wire Line
-	1200 4300 1300 4300
+	1450 3800 1550 3800
 $Comp
 L power1:GND #PWR03
 U 1 1 5950C2F7
-P 1300 4400
-F 0 "#PWR03" H 1300 4150 50  0001 C CNN
-F 1 "GND" H 1300 4250 50  0000 C CNN
-F 2 "" H 1300 4400 50  0001 C CNN
-F 3 "" H 1300 4400 50  0001 C CNN
-	1    1300 4400
-	1    0    0    -1
-$EndComp
-Wire Wire Line
-	1300 4300 1300 4400
-Connection ~ 1300 4300
-Wire Wire Line
-	1600 3900 1650 3900
-Wire Wire Line
-	1650 3900 1650 4000
-Wire Wire Line
-	1650 4000 1600 4000
+P 1550 3900
+F 0 "#PWR03" H 1550 3650 50  0001 C CNN
+F 1 "GND" H 1550 3750 50  0000 C CNN
+F 2 "" H 1550 3900 50  0001 C CNN
+F 3 "" H 1550 3900 50  0001 C CNN
+	1    1550 3900
+	1    0    0    -1
+$EndComp
+Wire Wire Line
+	1550 3800 1550 3900
 Wire Wire Line
 	5500 4850 6700 4850
@@
 NoConn ~ 4000 5450
 NoConn ~ 4000 5600
-NoConn ~ 5500 3950
-NoConn ~ 5500 4100
 NoConn ~ 5500 4250
 NoConn ~ 5500 5150
@@
 NoConn ~ 5500 5450
 NoConn ~ 5500 5600
-NoConn ~ 1600 4100
 Wire Wire Line
 	1350 2350 1350 2400
@@
 Wire Wire Line
 	6700 5000 7650 5000
+Text GLabel 5650 3950 2    60   Input ~ 0
+RX
+Text GLabel 5650 4100 2    60   Input ~ 0
+TX
+Wire Wire Line
+	5650 3950 5500 3950
+Wire Wire Line
+	5500 4100 5650 4100
+$Comp
+L Connector_Generic:Conn_01x02 J2
+U 1 1 5A9B6813
+P 1250 3800
+F 0 "J2" H 1170 3475 50  0000 C CNN
+F 1 "Conn_01x02" H 1170 3566 50  0000 C CNN
+F 2 "Connector_PinHeader_2.54mm:PinHeader_1x02_P2.54mm_Vertical" H 1250 3800 50  0001 C CNN
+F 3 "~" H 1250 3800 50  0001 C CNN
+	1    1250 3800
+	-1   0    0    1
+$EndComp
 $EndSCHEMATC

Commit message: actualizando todos los perifericos
Parts:
- removed C1: 10uF, Capacitors_SMD:CP_Elec_4x5.3, symbol omega-dock-new-rescue:CP_Small-RESCUE-omega-dock-new
- removed C2: 100uF, Capacitors_SMD:CP_Elec_6.3x5.3, symbol omega-dock-new-rescue:CP_Small-RESCUE-omega-dock-new
- removed J2: Conn_01x02, Connector_PinHeader_2.54mm:PinHeader_1x02_P2.54mm_Vertical, symbol Connector_Generic:Conn_01x02
- removed J3: RJ45-TRAFO, RJ45-TRAFO-AMPHENOL:RJ45_TRAFO_AMPHENOL, symbol omega-dock-new:RJ45-TRAFO
- removed U2: AP111733, TO_SOT_Packages_SMD:SOT-223, symbol omega-dock-new-rescue:AP111733-RESCUE-omega-dock-new
- added C4: 1nF, Capacitor_SMD:C_0805_2012Metric_Pad1.15x1.50mm_HandSolder, symbol Device:C
- added D1, D2, D3: LED, LED_SMD:LED_0805_2012Metric_Castellated, symbol Device:LED_ALT
- added J2: RJMG1BD3B8K1ANR, Devices_MSS:RJMG1B, symbol Mss_devices:RJMG1BD3B8K1ANR
- added L1: 220@100MHz, Inductor_SMD:L_0805_2012Metric_Pad1.15x1.50mm_HandSolder, symbol Device:L_Core_Ferrite_Small
- added R1, R2, R3: 220, Resistor_SMD:R_0805_2012Metric_Pad1.15x1.50mm_HandSolder, symbol Device:R
- C1: renamed from C3; footprint Capacitors_SMD:C_0805_HandSoldering -> Capacitor_SMD:C_0805_2012Metric_Pad1.15x1.50mm_HandSolder
- C2: renamed from C4; footprint Capacitors_SMD:C_0805_HandSoldering -> Capacitor_SMD:C_0805_2012Metric_Pad1.15x1.50mm_HandSolder
- C3: renamed from C5; value 1uF -> 47uF; footprint Capacitors_SMD:C_0805_HandSoldering -> Capacitor_Tantalum_SMD:CP_EIA-3528-12_Kemet-T_Pad1.63x2.40mm_HandSolder; symbol omega-dock-new-rescue:C-RESCUE-omega-dock-new -> Device:CP1
- D4: renamed from D1; footprint LEDs:LED_1206_HandSoldering -> LED_SMD:LED_0805_2012Metric_Castellated; symbol omega-dock-new-rescue:LED-RESCUE-omega-dock-new -> Device:LED_ALT
- F1: footprint Capacitors_SMD:C_1206_HandSoldering -> Capacitor_SMD:C_1206_3216Metric_Pad1.24x1.80mm_HandSolder
- J1: footprint Connectors:USB_A -> Connector_USB:USB_A_Horizontal
- R4: renamed from R2; footprint Resistors_SMD:R_0805_HandSoldering -> Resistor_SMD:R_0805_2012Metric_Pad1.15x1.50mm_HandSolder
- R5: renamed from R1; footprint Resistors_SMD:R_0805_HandSoldering -> Resistor_SMD:R_0805_2012Metric_Pad1.15x1.50mm_HandSolder
- R6: renamed from R3; footprint Resistors_SMD:R_0805_HandSoldering -> Resistor_SMD:R_0805_2012Metric_Pad1.15x1.50mm_HandSolder
- R7: renamed from R4; footprint Resistors_SMD:R_0805_HandSoldering -> Resistor_SMD:R_0805_2012Metric_Pad1.15x1.50mm_HandSolder
- R8: renamed from R5; footprint Resistors_SMD:R_0805_HandSoldering -> Resistor_SMD:R_0805_2012Metric_Pad1.15x1.50mm_HandSolder; symbol omega-dock-new-rescue:R-RESCUE-omega-dock-new -> Device:R
- U1: footprint TO_SOT_Packages_SMD:SOT-23-6_Handsoldering -> Package_TO_SOT_SMD:SOT-23-6_Handsoldering
- U2: renamed from U3; footprint (none) -> Devices_MSS:OMEGA_2
Connections:
- net labels added: GNDREF
- wire segments 79 -> 94
Other:
- moved on the sheet: C1, C2, R4, R5, R6, R7
